File: odrive.kicad_pcb (KiCad board)
At the start: 2 copper layers, 50 parts, among them J1 Conn_01x08_Female, J11 Conn_01x04_Female, J4 Barrel_Jack_Switch_Pin3Ring, Q1 PSMN020-100YS, Q2 PSMN020-100YS, Q3 PSMN020-100YS, Q4 PSMN020-100YS, Q5 PSMN020-100YS, Q6 PSMN010-100YS, U1 LM7805_TO220, U2 2EDL05, U3 2EDL05, U4 2EDL05, U5 tsv914a

Commit message: schematic complete. pcb routed
Parts:
- removed D1, D2, D3: D, Diode_SMD:D_0805_2012Metric_Pad1.15x1.40mm_HandSolder
- added J2: Conn_01x02, Connector_PinHeader_2.54mm:PinHeader_1x02_P2.54mm_Vertical, F.Cu at (260.9, 105.3)
- C7, C8, C9: moved to F.Cu
- moved C9 23.7 mm to (260.8, 85.4), turned to 0 degrees
- moved C8 20.6 mm to (260.9, 64.2), turned to 0 degrees
- moved R13 20.1 mm to (249.1, 100.6), turned to 180 degrees
- moved C5 19.6 mm to (250.7, 90.2)
- moved C6 19.5 mm to (248.2, 90.2)
- moved R12 18.8 mm to (249.1, 102.6), turned to 180 degrees
- moved R11 17.6 mm to (249.1, 105.1), turned to 180 degrees
- moved R10 17.2 mm to (249.1, 107.1), turned to 180 degrees
- moved J1 16.7 mm to (241.6, 66.0)
- moved C7 16.1 mm to (261.0, 44.2), turned to 0 degrees
- moved C10 15.9 mm to (242.1, 98.1), turned to 180 degrees
- moved J11 15.7 mm to (226.1, 105.9), turned to 180 degrees
- moved C3 15.7 mm to (250.0, 69.1)
- moved C4 15.6 mm to (247.6, 69.1)
- moved C11 13.4 mm to (242.1, 100.1), turned to 180 degrees
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Connections:
- C7 pad 1: Net-(C7-Pad1) -> VBUS
- C8 pad 1: Net-(C8-Pad1) -> VBUS
- C9 pad 1: Net-(C9-Pad1) -> VBUS
- J1 pad 3: Net-(J1-Pad3) -> Net-(U2-Pad2)
- J1 pad 4: Net-(J1-Pad4) -> Net-(U2-Pad3)
- U2 pad 2: Net-(J1-Pad4) -> Net-(U2-Pad2)
- U2 pad 3: Net-(J1-Pad3) -> Net-(U2-Pad3)
- U2 pad 8: Net-(C7-Pad1) -> VBUS
- U3 pad 2: Net-(J1-Pad6) -> Net-(J1-Pad5)
- U3 pad 3: Net-(J1-Pad5) -> Net-(J1-Pad6)
- U3 pad 8: Net-(C8-Pad1) -> VBUS
- U4 pad 2: Net-(J1-Pad8) -> Net-(J1-Pad7)
- U4 pad 3: Net-(J1-Pad7) -> Net-(J1-Pad8)
- U4 pad 8: Net-(C9-Pad1) -> VBUS
Routing:
- net Net-(Q2-Pad1): track 0.00 -> 87.4 mm, vias 0 -> 3
- net VBUS: track 51.0 -> 136.2 mm
- net VCC: track 53.7 -> 130.8 mm, vias 3 -> 5
- net GND: track 158.8 -> 233.4 mm, vias 15 -> 20
- net Net-(Q4-Pad1): track 0.00 -> 68.9 mm, vias 0 -> 5
- net +3V3: track 19.5 -> 68.1 mm, vias 0 -> 1
- net Net-(Q6-Pad1): track 0.00 -> 45.9 mm, vias 0 -> 4
- net Net-(J1-Pad4): track 34.2 -> 0.00 mm
- net Net-(J1-Pad3): track 33.3 -> 0.00 mm
- net Net-(U2-Pad3): track 0.00 -> 31.1 mm
- net Net-(U2-Pad2): track 0.00 -> 30.2 mm
- net Net-(J11-Pad2): track 3.99 -> 32.6 mm, vias 0 -> 2
- net /W: track 1.86 -> 25.8 mm, vias 1 -> 2
- net /V: track 1.86 -> 24.7 mm, vias 1 -> 2
- net /U: track 1.86 -> 24.6 mm, vias 1 -> 2
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- added copper zone on F.Cu, net Net-(Q2-Pad1)
- added copper zone on F.Cu, net Net-(Q4-Pad1)
- added copper zone on F.Cu, net Net-(Q6-Pad1)

Commit message: Add files via upload
Parts:
- added ?: , , F.Cu at (142.3, 92.7)
- added ?: , , F.Cu at (148.5, 116.7)
- added ?: , , F.Cu at (142.3, 107.0)
- added ?: , , F.Cu at (148.5, 145.2)
- added ?: , , F.Cu at (142.3, 102.3)
- added ?: , , F.Cu at (142.3, 121.2)
- added ?: , , F.Cu at (148.5, 92.9)
- added ?: , , F.Cu at (148.5, 121.4)
- added ?: , , F.Cu at (148.5, 102.5)
- added ?: , , F.Cu at (148.5, 107.1)
- added ?: , , F.Cu at (142.3, 116.6)
- added ?: , , F.Cu at (142.3, 135.5)
- added ?: , , F.Cu at (148.5, 131.0)
- added ?: , , F.Cu at (142.3, 130.8)
- added ?: , , F.Cu at (142.3, 145.1)
- added ?: , , F.Cu at (148.5, 135.6)
- added C1: 4.7U, Capacitor_SMD:C_0805_2012Metric_Pad1.18x1.45mm_HandSolder, B.Cu at (112.8, 142.0)
- added C10: 4.7U, Capacitor_SMD:C_0805_2012Metric_Pad1.18x1.45mm_HandSolder, F.Cu at (118.7, 92.9)
- added C11: 10n, Capacitor_SMD:C_0805_2012Metric_Pad1.18x1.45mm_HandSolder, F.Cu at (118.7, 90.9)
- added C2: 10n, Capacitor_SMD:C_0805_2012Metric_Pad1.18x1.45mm_HandSolder, B.Cu at (110.4, 142.0)
- added C3: 4.7U, Capacitor_SMD:C_0805_2012Metric_Pad1.18x1.45mm_HandSolder, B.Cu at (110.8, 121.9)
- added C4: 10n, Capacitor_SMD:C_0805_2012Metric_Pad1.18x1.45mm_HandSolder, B.Cu at (113.2, 122.0)
- added C5: 4.7U, Capacitor_SMD:C_0805_2012Metric_Pad1.18x1.45mm_HandSolder, B.Cu at (110.1, 100.8)
- added C6: 10n, Capacitor_SMD:C_0805_2012Metric_Pad1.18x1.45mm_HandSolder, B.Cu at (112.6, 100.8)
- added C7: 4.7u, Capacitor_SMD:C_1206_3216Metric_Pad1.33x1.80mm_HandSolder, F.Cu at (99.8, 147.5)
- added C8: 4.7u, Capacitor_SMD:C_1206_3216Metric_Pad1.33x1.80mm_HandSolder, F.Cu at (100.0, 127.4)
- added C9: 4.7u, Capacitor_SMD:C_1206_3216Metric_Pad1.33x1.80mm_HandSolder, F.Cu at (99.9, 106.7)
- added J1: Conn_01x08_Female, Connector_PinHeader_2.54mm:PinHeader_1x08_P2.54mm_Vertical, F.Cu at (119.2, 125.0)
- added J11: Conn_01x04_Female, Connector_PinHeader_2.54mm:PinHeader_1x04_P2.54mm_Vertical, F.Cu at (134.7, 85.1)
- added J2: Conn_01x02, Connector_PinHeader_2.54mm:PinHeader_1x02_P2.54mm_Vertical, F.Cu at (100.0, 85.7)
- added J3: Conn_01x08_Female, Connector_PinHeader_2.54mm:PinHeader_1x08_P2.54mm_Vertical, F.Cu at (122.3, 125.0)
- added J3: Conn_01x08_Female, Connector_PinHeader_2.54mm:PinHeader_1x08_P2.54mm_Vertical, F.Cu at (109.9, 64.3)
- added J4: Barrel_Jack_Switch_Pin3Ring, A_user:CUI_PJ-002BH-SMT-TR, F.Cu at (123.3, 137.1)
- added J5: Conn_01x04_Female, Connector_PinHeader_2.54mm:PinHeader_1x04_P2.54mm_Vertical, F.Cu at (131.9, 85.2)
- added J5: Conn_01x04_Female, Connector_PinHeader_2.54mm:PinHeader_1x04_P2.54mm_Vertical, F.Cu at (149.7, 73.9)
- added Q1: PSMN020-100YS, Package_TO_SOT_SMD:LFPAK56, F.Cu at (86.9, 141.5)
- added Q2: PSMN020-100YS, Package_TO_SOT_SMD:LFPAK56, F.Cu at (89.2, 147.2)
- added Q3: PSMN020-100YS, Package_TO_SOT_SMD:LFPAK56, F.Cu at (86.9, 121.3)
- added Q4: PSMN020-100YS, Package_TO_SOT_SMD:LFPAK56, F.Cu at (89.3, 127.0)
- added Q5: PSMN020-100YS, Package_TO_SOT_SMD:LFPAK56, F.Cu at (86.8, 100.3)
- added Q6: PSMN010-100YS, Package_TO_SOT_SMD:LFPAK56, F.Cu at (89.2, 106.0)
- added R1: 10m, Resistor_SMD:R_2512_6332Metric_Pad1.40x3.35mm_HandSolder, F.Cu at (93.8, 153.0)
- added R10: 10K, Resistor_SMD:R_0805_2012Metric_Pad1.20x1.40mm_HandSolder, F.Cu at (111.7, 83.9)
- added R11: 120, Resistor_SMD:R_0805_2012Metric_Pad1.20x1.40mm_HandSolder, F.Cu at (111.7, 85.9)
- added R12: 120, Resistor_SMD:R_0805_2012Metric_Pad1.20x1.40mm_HandSolder, F.Cu at (111.7, 88.4)
- added R13: 10K, Resistor_SMD:R_0805_2012Metric_Pad1.20x1.40mm_HandSolder, F.Cu at (111.7, 90.4)
- added R14: 10K, Resistor_SMD:R_0805_2012Metric_Pad1.20x1.40mm_HandSolder, F.Cu at (125.7, 83.4)
- added R15: 120, Resistor_SMD:R_0805_2012Metric_Pad1.20x1.40mm_HandSolder, F.Cu at (125.7, 85.4)
- added R16: 120, Resistor_SMD:R_0805_2012Metric_Pad1.20x1.40mm_HandSolder, F.Cu at (125.7, 87.9)
- added R17: 10K, Resistor_SMD:R_0805_2012Metric_Pad1.20x1.40mm_HandSolder, F.Cu at (125.7, 89.9)
- added R2: 10m, Resistor_SMD:R_2512_6332Metric_Pad1.40x3.35mm_HandSolder, F.Cu at (93.8, 133.0)
- added R3: 10m, Resistor_SMD:R_2512_6332Metric_Pad1.40x3.35mm_HandSolder, F.Cu at (93.8, 112.0)
- added R4: 100, Resistor_SMD:R_0805_2012Metric_Pad1.20x1.40mm_HandSolder, F.Cu at (95.8, 139.0)
- added R5: 100, Resistor_SMD:R_0805_2012Metric_Pad1.20x1.40mm_HandSolder, F.Cu at (95.8, 145.0)
- added R6: 100, Resistor_SMD:R_0805_2012Metric_Pad1.20x1.40mm_HandSolder, F.Cu at (95.8, 119.0)
- added R7: 100, Resistor_SMD:R_0805_2012Metric_Pad1.20x1.40mm_HandSolder, F.Cu at (95.8, 125.0)
- added R8: 100, Resistor_SMD:R_0805_2012Metric_Pad1.20x1.40mm_HandSolder, F.Cu at (95.8, 98.0)
- added R9: 100, Resistor_SMD:R_0805_2012Metric_Pad1.20x1.40mm_HandSolder, F.Cu at (95.8, 104.0)
- added REF**: sfp_1_port, 1_user:sfp_1_port, F.Cu at (161.7, 28.9)
- added REF**: sfp_2_port, 1_user:sfp_2_port, F.Cu at (160.4, 52.8)
- added REF**: sfp_4_port, 1_user:sfp_4_port, F.Cu at (160.0, 95.8)
- added U1: LM7805_TO220, Package_TO_SOT_THT:TO-220-3_Vertical, F.Cu at (126.5, 129.5)
- added U2: 2EDL05, Package_SO:SO-8_3.9x4.9mm_P1.27mm, F.Cu at (102.8, 142.0)
- added U3: 2EDL05, Package_SO:SO-8_3.9x4.9mm_P1.27mm, F.Cu at (102.8, 122.0)
- added U4: 2EDL05, Package_SO:SO-8_3.9x4.9mm_P1.27mm, F.Cu at (102.8, 100.8)
- added U5: tsv914a, Package_SO:TSSOP-14_4.4x5mm_P0.65mm, F.Cu at (118.7, 86.4)
- added U_1: Conn_01x01_Female, MountingHole:MountingHole_2.7mm_M2.5_DIN965_Pad, F.Cu at (81.8, 147.2)
- added VB+1: Conn_01x01_Female, MountingHole:MountingHole_2.7mm_M2.5_DIN965_Pad, F.Cu at (86.8, 91.0)
- added VB-1: Conn_01x01_Female, MountingHole:MountingHole_2.7mm_M2.5_DIN965_Pad, F.Cu at (93.8, 91.0)
- added V_1: Conn_01x01_Female, MountingHole:MountingHole_2.7mm_M2.5_DIN965_Pad, F.Cu at (81.8, 127.0)
- added W_1: Conn_01x01_Female, MountingHole:MountingHole_2.7mm_M2.5_DIN965_Pad, F.Cu at (81.9, 106.0)
- C7, C8, C9: value C -> 4.7u; footprint Capacitor_SMD:C_0805_2012Metric_Pad1.18x1.45mm_HandSolder -> Capacitor_SMD:C_1206_3216Metric_Pad1.33x1.80mm_HandSolder
- R4, R5, R6, R7, R8, R9: value R -> 100
- moved U_1 192.4 mm to (87.7, 23.8), turned to 90 degrees
- moved R1 185.1 mm to (81.9, 35.9), turned to -90 degrees
- moved Q2 184.4 mm to (87.7, 31.2), turned to 90 degrees
- moved Q1 181.8 mm to (93.4, 28.9), turned to 90 degrees
- moved V_1 175.8 mm to (107.9, 23.9), turned to 90 degrees
- moved R5 175.3 mm to (89.9, 37.9), turned to 90 degrees
- moved C7 173.7 mm to (87.4, 41.8), turned to 90 degrees
- moved R4 169.7 mm to (95.9, 37.9), turned to 90 degrees
- moved Q4 166.9 mm to (107.9, 31.3), turned to 90 degrees
- moved R2 166.6 mm to (101.9, 35.9), turned to -90 degrees
- moved Q3 165.5 mm to (113.6, 28.9), turned to 90 degrees
- moved U2 165.2 mm to (92.9, 44.9), turned to 90 degrees
- moved W_1 162.6 mm to (128.9, 23.9), turned to 90 degrees
- moved R7 157.7 mm to (109.9, 37.9), turned to 90 degrees
- moved C2 157.6 mm to (92.9, 52.4), turned to 0 degrees
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Connections:
- net Net-(Q2-Pad1) renamed /u_current
- net Net-(Q4-Pad1) renamed /v_current
- net Net-(Q6-Pad1) renamed /w_current
Routing:
- net GND: track 233.4 -> 466.9 mm, vias 20 -> 40
- net VBUS: track 136.2 -> 274.4 mm, vias 6 -> 12
- net VCC: track 130.8 -> 261.7 mm, vias 5 -> 10
- net /u_current: track 87.4 -> 174.8 mm, vias 3 -> 4
- net /v_current: track 68.9 -> 137.7 mm, vias 5 -> 8
- net +3V3: track 68.1 -> 136.2 mm, vias 1 -> 0
- net /w_current: track 45.9 -> 91.8 mm, vias 4 -> 8
- net Net-(J1-Pad4): track 31.1 -> 68.5 mm
- net Net-(J1-Pad3): track 30.2 -> 66.5 mm
- net Net-(J11-Pad2): track 32.6 -> 65.2 mm, vias 2 -> 4
- net Net-(J11-Pad1): track 25.7 -> 54.8 mm
- net /W: track 25.8 -> 50.6 mm, vias 2 -> 4
- net /V: track 24.7 -> 49.4 mm, vias 2 -> 4
- net /U: track 24.6 -> 49.2 mm, vias 2 -> 4
- net Net-(J11-Pad4): track 22.4 -> 46.8 mm, vias 1 -> 2
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