File: odrive.kicad_sch (KiCad schematic)
At the start: 50 parts, among them J1 Conn_01x08_Female, J11 Conn_01x04_Female, J4 Barrel_Jack_Switch_Pin3Ring, Q1 PSMN020-100YS, Q2 PSMN020-100YS, Q3 PSMN020-100YS, Q4 PSMN020-100YS, Q5 PSMN020-100YS, Q6 PSMN010-100YS, U1 LM7805_TO220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

Commit message: schematic complete. pcb routed
Parts:
- removed D1, D2, D3: D, Diode_SMD:D_0805_2012Metric_Pad1.15x1.40mm_HandSolder, symbol Device:D
- added J2: Conn_01x02, Connector_PinHeader_2.54mm:PinHeader_1x02_P2.54mm_Vertical, symbol Connector_Generic:Conn_01x02
Connections:
- net VBUS: now also C7.1, C8.1, C9.1, U2.8 (VBUS), U3.8 (VBUS), U4.8 (VBUS), J2.2 (Pin_2)
- net VCC: now also J2.1 (Pin_1)
- net at J1.3 (Pin_3): now also U2.2 (HIN); no longer U2.3 (LIN)
- net at J1.4 (Pin_4): now also U2.3 (LIN); no longer U2.2 (HIN)
- net at J1.5 (Pin_5): now also U3.2 (HIN); no longer U3.3 (LIN)
- net at J1.6 (Pin_6): now also U3.3 (LIN); no longer U3.2 (HIN)
- net at J1.7 (Pin_7): now also U4.2 (HIN); no longer U4.3 (LIN)
- net at J1.8 (Pin_8): now also U4.3 (LIN); no longer U4.2 (HIN)

Commit message: Add files via upload
Parts:
- added J3: Conn_01x08_Female, Connector_PinHeader_2.54mm:PinHeader_1x08_P2.54mm_Vertical, symbol Connector:Conn_01x08_Female
- added J5: Conn_01x04_Female, Connector_PinHeader_2.54mm:PinHeader_1x04_P2.54mm_Vertical, symbol Connector:Conn_01x04_Female
- C7, C8, C9: value C -> 4.7u; footprint Capacitor_SMD:C_0805_2012Metric_Pad1.18x1.45mm_HandSolder -> Capacitor_SMD:C_1206_3216Metric_Pad1.33x1.80mm_HandSolder
- R4, R5, R6, R7, R8, R9: value R -> 100
Connections:
- net +3V3: now also J3.1 (Pin_1)
- net GND: now also J3.2 (Pin_2)
- net u_current: now reaches Q2.1 (S), Q2.2 (S), Q2.3 (S), R1.2, U5.3 (a_in+)
- net v_current: now reaches Q4.1 (S), Q4.2 (S), Q4.3 (S), R2.2, U5.5 (b_in+)
- net at J1.3 (Pin_3), U2.2 (HIN): now also J3.3 (Pin_3)
- net at J1.4 (Pin_4), U2.3 (LIN): now also J3.4 (Pin_4)
- net at J1.5 (Pin_5), U3.2 (HIN): now also J3.5 (Pin_5)
- net at J1.6 (Pin_6), U3.3 (LIN): now also J3.6 (Pin_6)
- net at J1.7 (Pin_7), U4.2 (HIN): now also J3.7 (Pin_7)
- net at J1.8 (Pin_8), U4.3 (LIN): now also J3.8 (Pin_8)
- net at J11.3 (Pin_3), R17.2, U5.8 (c_out): now also J5.3 (Pin_3)
- net at J11.1 (Pin_1), R10.2, U5.1 (a_out): now also J5.1 (Pin_1)
- net w_current: now reaches Q6.1 (S), Q6.2 (S), Q6.3 (S), R3.2, U5.10 (c_in+)
- net at J11.4 (Pin_4), R14.2, U5.14 (d_out): now also J5.4 (Pin_4)
- net at J11.2 (Pin_2), R13.2, U5.7 (b_out): now also J5.2 (Pin_2)
